Commit message: feat: 测试多机器人

File: robot_model/sr5/sp_description/urdf/common_properties.xacro (robot description, xacro)
@@ -2,9 +2,9 @@
 <robot name="xacro_properties" xmlns:xacro="http://ros.org/wiki/xacro">
   <xacro:property name="M_PI" value="3.1415926535897931" />
-  <macro name="cylinder_inertia" params="m r h">
+  <!--macro name="cylinder_inertia" params="m r h">
     <inertia  ixx="${m*(3*r*r+h*h)/12}" ixy = "0" ixz = "0"
               iyy="${m*(3*r*r+h*h)/12}" iyz = "0"
               izz="${m*r*r/2}" />
-  </macro>
+  </macro-->
   <!-- Init colour -->
   <material name="black">

File: robot_model/sr5/sp_description/urdf/sr7e/sr7e.urdf.xacro (robot description, xacro)
@@ -9,7 +9,7 @@
   <xacro:property name="height" value="0.20" /> <!-- base link height -->
   <!-- Wheels -->
-  <property name="wheel_radius" value="0.076" />
-  <property name="wheel_height" value="0.02" />
-  <property name="wheel_mass" value="2.50" /> <!-- in kg-->
+  <xacro:property name="wheel_radius" value="0.076" />
+  <xacro:property name="wheel_height" value="0.02" />
+  <xacro:property name="wheel_mass" value="2.50" /> <!-- in kg-->
   <link name="base_footprint"/>
   <joint name="base_joint" type="fixed">
@@ -23,5 +23,4 @@
       <origin xyz="0 0 0.01" rpy="0 0 0"/>
       <geometry>
-	      <!--box size="${width} ${width} ${height}"/-->
 	      <box size="0.40 0.40 0.02"/>
       </geometry>
@@ -31,7 +30,5 @@
       <origin xyz="0 0 0.01" rpy="0 0 0"/>
       <geometry>
-	      <!--box size="0.40 0.40 0.02"/-->
-	      <!--box size="${width} ${width} ${height}"/-->
-        <!--mesh filename="package://sp_gazebo/meshes/AMR.STL" scale="0.001 0.001 0.001"/-->
+	      <box size="0.40 0.40 0.02"/>
       </geometry>
       <material name="white"/>
@@ -184,13 +181,13 @@
   <!-- caster wheel radius and height -->
   <!-- caster wheel mass -->
-  <property name="caster_f_height" value="0.00" />
-  <property name="caster_f_radius" value="0.025" />
-  <property name="caster_f_mass" value="5.0" /> <!-- in kg-->
-  <property name="caster_height" value="-0.029" />
+  <xacro:property name="caster_f_height" value="0.00" />
+  <xacro:property name="caster_f_radius" value="0.025" />
+  <xacro:property name="caster_f_mass" value="5.0" /> <!-- in kg-->
+  <xacro:property name="caster_height" value="-0.029" />
   <!-- caster wheel radius and height -->
   <!-- caster wheel mass -->
-  <property name="caster_b_height" value="0.00" />
-  <property name="caster_b_radius" value="0.025" />
-  <property name="caster_b_mass" value="5.0" /> <!-- in kg-->
+  <xacro:property name="caster_b_height" value="0.00" />
+  <xacro:property name="caster_b_radius" value="0.025" />
+  <xacro:property name="caster_b_mass" value="5.0" /> <!-- in kg-->
 <!--Caster front  -->
   <joint name="caster_front_left_joint" type="fixed">
